File: bloo.kicad_pcb (KiCad board)
At the start: 2 copper layers, 90 x 96 mm, 95 parts, among them J5 SWD_Header, M1 M1_Conn_Alt, M2 M2_Conn_Alt, Q0 TEFT4300, Q1 TEFT4300, Q10 Q_NMOS_GSD, Q11 Q_NMOS_GSD, Q12 Q_NMOS_GSD, Q2 TEFT4300, Q3 TEFT4300, Q9 Q_NMOS_GSD, U1 YAAJ_BluePill_SWD_Breakout, U2 L293D, U3 LM1085-5.0, U4 NCP161ASN330T1G, U5 BC832, Y1 ABS07-32.768KHZ-T

Commit message: prepare the layout file
Parts:
- removed BT1: Battery_Cell, Connector_AMASS:AMASS_XT30UPB-M_1x02_P5.0mm_Vertical
- removed BT_MH1, BT_MH2, BT_MH3, BT_MH4, SK1, SK2, SK3, SK4: M2, MountingHole:MountingHole_2.2mm_M2
- removed C1, C12, C13, C19, C22, C4: 0.1uF, Capacitor_SMD:C_1206_3216Metric_Pad1.33x1.80mm_HandSolder
- removed C10: 10uF(Tantalum), Capacitor_SMD:C_1206_3216Metric_Pad1.33x1.80mm_HandSolder
- removed C11, C9: 10uF, Capacitor_SMD:C_1206_3216Metric_Pad1.33x1.80mm_HandSolder
- removed C14, C15, C17, C18, C20, C21, C3: 1uF, Capacitor_SMD:C_1206_3216Metric_Pad1.33x1.80mm_HandSolder
- removed C16, C2: 100uF, Capacitor_THT:CP_Radial_D6.3mm_P2.50mm
- removed C25: 10nF, Capacitor_SMD:C_1206_3216Metric_Pad1.33x1.80mm_HandSolder
- removed C5: 100nF, Capacitor_SMD:C_0603_1608Metric
- removed C6: 47µF, Capacitor_SMD:C_1206_3216Metric
- removed C7, C8: 12pF, Capacitor_SMD:C_0603_1608Metric_Pad1.08x0.95mm_HandSolder
- removed D0, D1, D2, D3: SFH4545, MM_Library:Emitter
- removed D4, D5, D6: LED, LED_SMD:LED_0805_2012Metric_Pad1.15x1.40mm_HandSolder
- removed D7, D9: 1SS389,L3F, Diode_SMD:D_SOD-523
- removed G***: LOGO, LOGO
- removed J5: SWD_Header, Connector_PinHeader_2.54mm:PinHeader_1x05_P2.54mm_Vertical
- removed JP4: Jumper_2_Open, Jumper:SolderJumper-2_P1.3mm_Bridged_Pad1.0x1.5mm
- removed L1: 10uH, Inductor_SMD:L_1206_3216Metric_Pad1.42x1.75mm_HandSolder
- removed M1: M1_Conn_Alt, Connector_JST:JST_SH_BM06B-SRSS-TB_1x06-1MP_P1.00mm_Vertical
- removed M2: M2_Conn_Alt, Connector_JST:JST_SH_BM06B-SRSS-TB_1x06-1MP_P1.00mm_Vertical
- removed M_MH1, M_MH2: M2, MM_Library:Motor_mouse
- removed Q0, Q1, Q2, Q3: TEFT4300, MM_Library:Emitter
- removed Q10, Q11, Q12, Q9: Q_NMOS_GSD, Package_TO_SOT_SMD:SOT-23
- removed R1, R2, R3, R4: 1.8K, Resistor_SMD:R_1206_3216Metric_Pad1.30x1.75mm_HandSolder
- removed R10, R23: 10K, Resistor_SMD:R_1206_3216Metric_Pad1.30x1.75mm_HandSolder
- removed R12, R13, R14, R15, R16, R17, R24, R9: 47K, Resistor_SMD:R_1206_3216Metric_Pad1.30x1.75mm_HandSolder
- removed R19: 750, Resistor_SMD:R_1206_3216Metric_Pad1.30x1.75mm_HandSolder
- removed R20, R21: 75, Resistor_SMD:R_1206_3216Metric_Pad1.30x1.75mm_HandSolder
- removed R22: 20K, Resistor_SMD:R_1206_3216Metric_Pad1.30x1.75mm_HandSolder
- removed R5, R6, R7, R8: 36, Resistor_SMD:R_1206_3216Metric_Pad1.30x1.75mm_HandSolder
- removed S1: EG1218, MM_Library:MM Switch
- removed S2, S3, S5: SKRPABE010, MM_Library:SW4_SKRPABE010_ALPS
- removed TP1: V_EXT_TP, Connector_PinHeader_2.54mm:PinHeader_1x01_P2.54mm_Vertical
- removed TP2, TP5, TP6: GND_TP, Connector_PinHeader_2.54mm:PinHeader_1x01_P2.54mm_Vertical
- removed TP3: TP_5V, Connector_PinHeader_2.54mm:PinHeader_1x01_P2.54mm_Vertical
- removed TP4: TP_3V3, Connector_PinHeader_2.54mm:PinHeader_1x01_P2.54mm_Vertical
- removed U1: YAAJ_BluePill_SWD_Breakout, MM_Library:STM32F103
- removed U2: L293D, Package_DIP:DIP-16_W7.62mm
- removed U3: LM1085-5.0, MM_Library:5V Voltage Reg
- removed U4: NCP161ASN330T1G, Package_TO_SOT_SMD:SOT-23-5
- removed U5: BC832, MM_Library:XCVR_BC832
- removed Y1: ABS07-32.768KHZ-T, MM_Library:CAP_ABS07-32.768KHZ-T_ABR
Routing:
- net +5V: track 242.3 -> 0.00 mm, vias 2 -> 0
- net +3V3: track 234.8 -> 0.00 mm, vias 1 -> 0
- net VCC: track 172.5 -> 0.00 mm, vias 3 -> 0
- net +3.3VA: track 123.3 -> 0.00 mm, vias 2 -> 0
- net BLE_SPI_MOSI: track 120.4 -> 0.00 mm, vias 7 -> 0
- net AGND: track 117.1 -> 0.00 mm, vias 8 -> 0
- net M1_ENC_A: track 113.1 -> 0.00 mm, vias 4 -> 0
- net BLE_SPI_SCK: track 106.6 -> 0.00 mm, vias 3 -> 0
- net BLE_LED: track 106.3 -> 0.00 mm, vias 5 -> 0
- net BLE_SPI_MISO: track 105.5 -> 0.00 mm, vias 4 -> 0
- net USART1_TX: track 103.0 -> 0.00 mm, vias 2 -> 0
- net M2_SPD: track 99.6 -> 0.00 mm, vias 1 -> 0
- net USART1_RX: track 98.0 -> 0.00 mm, vias 2 -> 0
- net M2_BACK: track 93.4 -> 0.00 mm, vias 1 -> 0
- net EMIT_4: track 91.5 -> 0.00 mm, vias 1 -> 0
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- removed copper zone on B.Cu, net GND
- removed copper zone on F.Cu, net GND
Other:
- board outline removed
- board text removed: "+"
- board text removed: "3V3"
- board text removed: "5V"
- board text removed: "Buttons"
- board text removed: "Emitters"
- board text removed: "GND"
- board text removed: "JMP"
- board text removed: "Receivers"
- board text removed: "VIN"
